File: AKS.kicad_pcb (KiCad board)
At the start: 2 copper layers, 29 x 63.5 mm, 13 parts, among them J1 Power, J10 JETSON_CAN, J2 Relay board, J3 JETSON DC JACK, J4 Jetson 40-pin GPIO, J5 BTS7960 H-bridge (signals onl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, J9 VESC_CAN, U1 SN65HVD230, U2 Polulu D24V10F5 (12 to 5V con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

Commit message: Add files via upload
Parts:
- moved C2 1.00 mm to (90.0, 117.0)
Routing:
- net /+12V_SAFE: track 35.9 -> 25.4 mm
- net /GND: track 69.6 -> 62.9 mm, vias 0 -> 4
- net /+3V3: track 77.9 -> 74.3 mm, vias 0 -> 1
- net /+12V: track 6.19 -> 7.43 mm
Other:
- board size 29 x 63.5 mm -> 29 x 63.9 mm
Changed lines of the file:
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@@
 		(capping no)
 		(filling no)
+		(zone_defaults)
 		(pcbplotparams
 			(layerselection 0x00000000_00000000_55555555_5755f5ff)
@@
 	(footprint "Capacitor_SMD:C_0805_2012Metric"
 		(layer "F.Cu")
-		(at 91 117)
+		(at 90 117)
 		(descr "Capacitor SMD 0805 (2012 Metric), square (rectangular) end terminal, IPC-7351 nominal, (Body size source: IPC-SM-782 page 76, https://www.pcb-3d.com/wordpress/wp-content/uploads/ipc-sm-782a_amendment_1_and_2.pdf, https://docs.google.com/spreadsheets/d/1BsfQQcO9C6DZCsRaXUlFlo91Tg2WpOkGARC1WS5S8t0/edit?usp=sharing)")
 		(tags "capacitor")
@@
 	)
 	(gr_rect
-		(start 71.45 97.95)
+		(start 71.45 97.5)
 		(end 100.45 161.45)
 		(stroke
@@
 	)
 	(segment
-		(start 91.905 101.95)
-		(end 91.45 101.495)
+		(start 95.5 100)
+		(end 92.945 100)
 		(width 2.5)
 		(layer "F.Cu")
@@
 	(segment
 		(start 97.45 101.95)
-		(end 91.905 101.95)
+		(end 95.5 100)
 		(width 2.5)
 		(layer "F.Cu")
@@
 	)
 	(segment
-		(start 91.45 106.405)
-		(end 90.865 106.99)
-		(width 2)
-		(layer "F.Cu")
-		(net "/+12V_SAFE")
-	)
-	(segment
-		(start 86.627308 116)
-		(end 89.05 116)
-		(width 0.5)
+		(start 92.945 100)
+		(end 91.45 101.495)
+		(width 2.5)
 		(layer "F.Cu")
-		(net "/+12V_SAFE")
+		(net "/+12V")
 	)
 	(segment
-		(start 85.237308 106.99)
-		(end 83.65 108.577308)
-		(width 0.5)
+		(start 91.45 106.405)
+		(end 90.865 106.99)
+		(width 2.5)
 		(layer "F.Cu")
 		(net "/+12V_SAFE")
@@
 		(start 90.865 106.99)
 		(end 85.95 106.99)
-		(width 0.75)
+		(width 2.5)
 		(layer "F.Cu")
 		(net "/+12V_SAFE")
 	)
 	(segment
-		(start 89.05 116)
-		(end 90 116.95)
-		(width 0.5)
+		(start 89.3 108.555)
+		(end 90.865 106.99)
+		(width 2.5)
 		(layer "F.Cu")
 		(net "/+12V_SAFE")
@@
 		(start 93.405 106.405)
 		(end 97.45 110.45)
-		(width 2)
+		(width 2.5)
 		(layer "F.Cu")
 		(net "/+12V_SAFE")
 	)
 	(segment
-		(start 89.3 109.137919)
-		(end 87.152081 106.99)
-		(width 2)
+		(start 89.3 111.95)
+		(end 89.3 108.555)
+		(width 2.5)
 		(layer "F.Cu")
 		(net "/+12V_SAFE")
 	)
 	(segment
-		(start 90 116.95)
-		(end 90 117)
+		(start 89 113.5)
+		(end 89 117)
 		(width 0.5)
 		(layer "F.Cu")
@@
 	)
 	(segment
-		(start 83.65 113.022692)
-		(end 86.627308 116)
+		(start 89.3 113.2)
+		(end 89.3 111.95)
 		(width 0.5)
 		(layer "F.Cu")
@@
 	)
 	(segment
-		(start 89.3 111.95)
-		(end 89.3 109.137919)
-		(width 2)
-		(layer "F.Cu")
-		(net "/+12V_SAFE")
-	)
-	(segment
 		(start 87.152081 106.99)
 		(end 85.95 106.99)
@@
 		(start 91.45 106.405)
 		(end 93.405 106.405)
-		(width 2)
-		(layer "F.Cu")
-		(net "/+12V_SAFE")
-	)
-	(segment
-		(start 85.95 106.99)
-		(end 85.237308 106.99)
-		(width 0.5)
+		(width 2.5)
 		(layer "F.Cu")
 		(net "/+12V_SAFE")
 	)
 	(segment
-		(start 83.65 108.577308)
-		(end 83.65 113.022692)
+		(start 89.3 113.2)
+		(end 89 113.5)
 		(width 0.5)
 		(layer "F.Cu")
@@
 		(start 84.45 153.19)
 		(end 85.95 154.69)
-		(width 0.5)
+		(width 0.75)
 		(layer "B.Cu")
 		(net "/+5V")
@@
 		(start 84.45 103.41)
 		(end 84.45 153.19)
-		(width 0.5)
+		(width 0.75)
 		(layer "B.Cu")
 		(net "/+5V")
@@
 		(start 85.95 101.91)
 		(end 84.45 103.41)
-		(width 0.5)
+		(width 0.75)
 		(layer "B.Cu")
 		(net "/+5V")
@@
 	)
 	(segment
-		(start 93.6 111.95)
-		(end 93.6 112.1)
-		(width 2)
-		(layer "F.Cu")
-		(net "/GND")
-	)
-	(segment
 		(start 92.41 139.064448)
 		(end 92.41 132.894448)
@@
 	)
 	(segment
-		(start 91.95 117)
-		(end 95.96 112.99)
-		(width 0.5)
-		(layer "F.Cu")
-		(net "/GND")
-	)
-	(segment
 		(start 95.62 142.998896)
 		(end 95.879448 142.739448)
@@
 	)
 	(segment
-		(start 94.95 113.45)
-		(end 96.99 113.45)
-		(width 2)
-		(layer "F.Cu")
-		(net "/GND")
-	)
-	(segment
 		(start 92.41 132.894448)
 		(end 93.265 132.039448)
@@
 	)
 	(segment
-		(start 96.99 113.45)
-		(end 97.45 112.99)
-		(width 2)
+		(start 90.95 118.45)
+		(end 91 118.5)
+		(width 0.2)
+		(layer "F.Cu")
+		(net "/GND")
+	)
+	(segment
+		(start 90.95 117)
+		(end 90.95 118.45)
+		(width 0.5)
 		(layer "F.Cu")
 		(net "/GND")
@@
 	)
 	(segment
-		(start 93.6 112.1)
-		(end 94.95 113.45)
-		(width 2)
-		(layer "F.Cu")
-		(net "/GND")
-	)
-	(segment
 		(start 92.41 139.064448)
 		(end 92.41 140.039447)
@@
 	)
 	(segment
-		(start 95.96 112.99)
-		(end 97.45 112.99)
-		(width 0.5)
+		(start 90.95 117)
+		(end 91.45 116.5)
+		(width 0.2)
 		(layer "F.Cu")
 		(net "/GND")
 	)
 	(segment
+		(start 93.6 111.95)
+		(end 93.6 114.9)
+		(width 2.5)
+		(layer "F.Cu")
+		(net "/GND")
+	)
+	(via
+		(at 93 115.5)
+		(size 0.8)
+		(drill 0.4)
+		(layers "F.Cu" "B.Cu")
+		(net "/GND")
+	)
+	(via
+		(at 94 115.5)
+		(size 0.8)
+		(drill 0.4)
+		(layers "F.Cu" "B.Cu")
+		(net "/GND")
+	)
+	(via
+		(at 91 118.5)
+		(size 0.7)
+		(drill 0.3)
+		(layers "F.Cu" "B.Cu")
+		(net "/GND")
+	)
+	(via
+		(at 93.6 114.9)
+		(size 0.8)
+		(drill 0.4)
+		(layers "F.Cu" "B.Cu")
+		(net "/GND")
+	)
+	(segment
 		(start 98.465 153.429448)
 		(end 97.315 154.579448)
@@
 	)
 	(segment
-		(start 91.365 132.039448)
-		(end 91.365 123.678654)
-		(width 0.2)
-		(layer "F.Cu")
-		(net "/+3V3")
-	)
-	(segment
 		(start 91.45 151.91)
 		(end 91.45 132.124448)
@@
 	)
 	(segment
-		(start 92.39 131.014448)
-		(end 91.365 132.039448)
+		(start 91.365 123.678654)
+		(end 79.731346 112.045)
 		(width 0.2)
 		(layer "F.Cu")
@@
 	)
 	(segment
-		(start 94.95 144.014448)
-		(end 94.95 141.95)
+		(start 94.95 142.05)
+		(end 95 142)
 		(width 0.2)
 		(layer "F.Cu")
@@
 	)
 	(segment
-		(start 94.95 141.95)
-		(end 93.08 140.08)
-		(width 0.2)
-		(layer "F.Cu")
-		(net "/+3V3")
-	)
-	(segment
-		(start 93.749744 131.014448)
-		(end 92.39 131.014448)
+		(start 77.865 106.965)
+		(end 76.69 105.79)
 		(width 0.2)
 		(layer "F.Cu")
@@
 	)
 	(segment
-		(start 93.08 140.08)
-		(end 93.08 137.578896)
+		(start 77.865 111.166701)
+		(end 77.865 106.965)
 		(width 0.2)
 		(layer "F.Cu")
@@
 	)
 	(segment
-		(start 91.365 123.678654)
-		(end 79.706346 112.02)
+		(start 78.743299 112.045)
+		(end 77.865 111.166701)
 		(width 0.2)
 		(layer "F.Cu")
@@
 	)
 	(segment
-		(start 94.065 136.593896)
-		(end 94.065 131.329704)
+		(start 79.731346 112.045)
+		(end 78.743299 112.045)
 		(width 0.2)
 		(layer "F.Cu")
@@
 	)
 	(segment
-		(start 79.706346 112.02)
-		(end 78.753654 112.02)
-		(width 0.2)
-		(layer "F.Cu")
-		(net "/+3V3")
-	)
-	(segment
-		(start 93.08 137.578896)
-		(end 94.065 136.593896)
+		(start 91.365 132.039448)
+		(end 91.365 123.678654)
 		(width 0.2)
 		(layer "F.Cu")
@@
 	)
 	(segment
-		(start 94.065 131.329704)
-		(end 93.749744 131.014448)
+		(start 94.95 144.014448)
+		(end 94.95 142.05)
 		(width 0.2)
 		(layer "F.Cu")
 		(net "/+3V3")
 	)
-	(segment
-		(start 78.753654 112.02)
-		(end 77.95 111.216346)
-		(width 0.2)
-		(layer "F.Cu")
+	(via
+		(at 95 142)
+		(size 0.6)
+		(drill 0.3)
+		(layers "F.Cu" "B.Cu")
 		(net "/+3V3")
 	)
 	(segment
-		(start 77.95 107.05)
-		(end 76.69 105.79)
-		(width 0.2)
-		(layer "F.Cu")
+		(start 91.45 145.55)
+		(end 91.45 151.91)
+		(width 0.25)
+		(layer "B.Cu")
 		(net "/+3V3")
 	)
 	(segment
-		(start 77.95 111.216346)
-		(end 77.95 107.05)
-		(width 0.2)
-		(layer "F.Cu")
+		(start 95 142)
+		(end 91.45 145.55)
+		(width 0.25)
+		(layer "B.Cu")
 		(net "/+3V3")
 	)
@@
 		(polygon
 			(pts
-				(xy 71.45 97.95) (xy 100.45 97.95) (xy 100.45 161.45) (xy 71.45 161.45)
+				(xy 71.45 97.5) (xy 100.45 97.5) (xy 100.45 161.45) (xy 71.45 161.45)
 			)
 		)
